Commit message: lower limit prevents gripper from over extending

File: robots/LoCoBot/locobot_description/urdf/interbotix_locobot_description.urdf (robot description, URDF)
Before this commit: robot locobot, 26 links, 25 joints
Joints:
- joint joint_6: limit lower=-1 upper=0 effort=1 velocity=1 -> lower=-0.033 upper=0 effort=100 velocity=50
- joint joint_7: limit lower=0 upper=1 effort=1 velocity=1 -> lower=0 upper=0.033 effort=100 velocity=50
