Commit message: Added camera dummy link to resolve point cloud orientation issue

File: robots/LoCoBot/locobot_description/urdf/locobot_description.urdf (robot description, URDF)
Before this commit: robot locobot, 26 links, 25 joints
Links:
- added link kinect_optical_link, mass 1e-5; collision box size=0.02 0.02 0.02; visual box size=0.1 0.1 0.1
Joints:
- added joint kinect_optical_joint: type fixed, parent camera_link, child kinect_optical_link, origin xyz=0.0 0.0 0.0 rpy=-1.57 0 -1.57, axis 0 1 0

Commit message: Resolved collision and visial issue with optical link

File: robots/LoCoBot/locobot_description/urdf/locobot_description.urdf (robot description, URDF)
Before this commit: robot locobot, 27 links, 26 joints
Links:
- link kinect_optical_link: geometry 
